File: symlib/symlib.kicad_sch (KiCad schematic)
At the start: 5 parts

Commit message: v0.1.0
Parts:
- removed -A17: X1.3, symbol plc_standart:PLC_OUT_(A)
- removed -B1: ~, symbol plc_standart:PNP Fe
- removed -K2: ~, symbol plc_standart:Relais (K)
- removed -K3: ~, symbol plc_standart:Relais_(K)_NC
- removed -X1: ~, symbol plc_standart:TCP_(X)
- added -K1, -K2: ~, symbol STD:Relais_(K)_NO
